Commit message: change xml

File: urdf/atom01.urdf (robot description, URDF)
Before this commit: robot atom01urdf, 25 links, 24 joints
Joints:
- joint right_ankle_roll_joint: limit lower=-0.5 upper=0.5 effort=18 velocity=3.7692 -> lower=-0.18 upper=0.18 effort=18 velocity=3.7692

Commit message: change urdf yaw axis

File: urdf/atom01.urdf (robot description, URDF)
Before this commit: robot atom01urdf, 25 links, 24 joints
Joints:
- joint right_arm_yaw_joint: axis 0 0 -1 -> 0 0 1

Commit message: V1.0_final version

File: urdf/atom01.urdf (robot description, URDF)
Before this commit: robot atom01urdf, 25 links, 24 joints
Links:
- removed link world
Joints:
- removed joint floating_base_joint
- joint left_ankle_roll_joint: limit lower=-0.18 upper=0.18 effort=18 velocity=3.7692 -> lower=-0.5 upper=0.5 effort=18 velocity=3.7692
- joint left_elbow_yaw_joint: axis 1 0 0 -> -1 0 0
- joint left_thigh_yaw_joint: axis 0.5 0 0.86603 -> -0.5 0 -0.86603; limit lower=-0.2 upper=1 effort=80 velocity=10.47 -> lower=-1 upper=0.2 effort=80 velocity=10.47
- joint right_ankle_roll_joint: limit lower=-0.18 upper=0.18 effort=18 velocity=3.7692 -> lower=-0.5 upper=0.5 effort=18 velocity=3.7692
- joint right_elbow_pitch_joint: limit lower=-1.5 upper=1.57 effort=18 velocity=3.7692 -> lower=-1.0 upper=1.57 effort=18 velocity=3.7692
- joint right_elbow_yaw_joint: axis 1 0 0 -> -1 0 0
- joint right_thigh_yaw_joint: axis 0.5 0 0.86603 -> -0.5 0 -0.86603; limit lower=-1 upper=0.2 effort=80 velocity=10.47 -> lower=-0.2 upper=1 effort=80 velocity=10.47
